Commit message: last_commit

File: ros2_ws/src/marl/urdf/robot.urdf (robot description, URDF)
Before this commit: robot swarm_robot, 7 links, 6 joints
Joints:
- removed joint left_wheel_joint
- removed joint right_wheel_joint
- added joint left_joint: type continuous, parent base_link, child left_wheel, origin xyz=0 0.06 0.02 rpy=0 0 0, axis 0 1 0
- added joint right_joint: type continuous, parent base_link, child right_wheel, origin xyz=0 -0.06 0.02 rpy=0 0 0, axis 0 -1 0
